Commit message: create contrllor by moveit

File: mycobot_description/urdf/mycobot_280_gripper/mycobot_with_gripper_parallel.urdf (robot description, URDF)
Before this commit: robot firefighter, 15 links, 14 joints
Links:
- link g_base: geometry collision mesh filename=package://mycobot_description/urdf/mycobot_280_gripper/G_ba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; visual mesh filename=package://mycobot_description/urdf/mycobot_280_gripper/G_ba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
- link gripper_base: geometry collision mesh filename=package://mycobot_description/urdf/mycobot_280_gripper/grip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; visual mesh filename=package://mycobot_description/urdf/mycobot_280_gripper/grip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
- link gripper_left1: geometry collision mesh filename=package://mycobot_description/urdf/mycobot_280_gripper/grip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; visual mesh filename=package://mycobot_description/urdf/mycobot_280_gripper/grip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
- link gripper_left2: geometry collision mesh filename=package://mycobot_description/urdf/mycobot_280_gripper/grip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; visual mesh filename=package://mycobot_description/urdf/mycobot_280_gripper/grip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
- link gripper_left3: geometry collision mesh filename=package://mycobot_description/urdf/mycobot_280_gripper/grip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; visual mesh filename=package://mycobot_description/urdf/mycobot_280_gripper/grip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
- link gripper_right1: geometry collision mesh filename=package://mycobot_description/urdf/mycobot_280_gripper/grip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; visual mesh filename=package://mycobot_description/urdf/mycobot_280_gripper/grip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
- link gripper_right2: geometry collision mesh filename=package://mycobot_description/urdf/mycobot_280_gripper/grip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; visual mesh filename=package://mycobot_description/urdf/mycobot_280_gripper/grip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
- link gripper_right3: geometry collision mesh filename=package://mycobot_description/urdf/mycobot_280_gripper/grip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; visual mesh filename=package://mycobot_description/urdf/mycobot_280_gripper/grip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
- link joint1: geometry collision mesh filename=package://mycobot_description/urdf/mycobot_280_gripper/join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; visual mesh filename=package://mycobot_description/urdf/mycobot_280_gripper/join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
- link joint2: geometry collision mesh filename=package://mycobot_description/urdf/mycobot_280_gripper/join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; visual mesh filename=package://mycobot_description/urdf/mycobot_280_gripper/join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
- link joint3: geometry collision mesh filename=package://mycobot_description/urdf/mycobot_280_gripper/join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; visual mesh filename=package://mycobot_description/urdf/mycobot_280_gripper/join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
- link joint4: geometry collision mesh filename=package://mycobot_description/urdf/mycobot_280_gripper/join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; visual mesh filename=package://mycobot_description/urdf/mycobot_280_gripper/join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
- link joint5: geometry collision mesh filename=package://mycobot_description/urdf/mycobot_280_gripper/join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; visual mesh filename=package://mycobot_description/urdf/mycobot_280_gripper/join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
- link joint6: geometry collision mesh filename=package://mycobot_description/urdf/mycobot_280_gripper/join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; visual mesh filename=package://mycobot_description/urdf/mycobot_280_gripper/join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
- link joint6_flange: geometry collision mesh filename=package://mycobot_description/urdf/mycobot_280_gripper/join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; visual mesh filename=package://mycobot_description/urdf/mycobot_280_gripper/join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
